File: KATO_FR11/board.brd (EAGLE design)
At the start: 12 x 8 mm, 15 parts, among them U2 ATTiny85

Commit message: Update with Routing
Parts:
- moved D4 4.71 mm to (8.30, 2.00), turned to 270 degrees
- moved D3 4.64 mm to (8.30, 3.40), turned to 90 degrees
- moved D2 3.10 mm to (3.70, 1.90)
- moved C2 2.98 mm to (5.45, 2.50), turned to 90 degrees
- moved D1 2.60 mm to (3.70, 3.40)
- moved Q1 2.55 mm to (5.40, 5.70), turned to 270 degrees
- moved R2 2.40 mm to (3.15, 5.80), flipped to the top
- moved U1 2.15 mm to (7.85, 5.70), turned to 270 degrees
- moved C1 1.49 mm to (6.55, 2.50)
- moved R1 1.27 mm to (3.15, 3.10), flipped to the top, turned to 90 degrees
- moved U2 0.32 mm to (6.30, 4.50)
Routing:
- net N$5: track 0.00 -> 7.53 mm, vias 0 -> 1
- net N$10: track 0.00 -> 7.37 mm, vias 0 -> 2
- net XT1: track 1.00 -> 8.13 mm, vias 0 -> 1
- net VIN: track 7.50 -> 14.3 mm, vias 1 -> 2
- net N$3: track 0.00 -> 4.92 mm
- net N$4: track 9.15 -> 4.85 mm
- net XT2: track 0.00 -> 3.70 mm
- net GND: track 0.00 -> 3.49 mm, vias 0 -> 1
- net N$1: track 0.00 -> 3.26 mm
- removed copper zone on layer 1, net GND
